File: mark-one/RAM.sch (KiCad schematic (older format))
At the start: 25 parts, among them P3 TST, U2 MX53, U4 MT41K256M16HA

Commit message: made changes
Parts:
- C100, C101, C102, C103, C104, C105, C106, C89, C90, C91, C93, C94, C95, C96, C97, C98, C99: symbol C -> armory-rescue:C
- P3: symbol TST -> armory-rescue:TST
- R15, R24, R27, R29, R30: symbol R -> armory-rescue:R
- U2: symbol MX53 -> armory:MX53
- U4: symbol MT41J256M16HA -> armory:MT41J256M16HA
Changed lines of the file:
@@
-EESchema Schematic File Version 2
-LIBS:power
-LIBS:device
-LIBS:transistors
-LIBS:conn
-LIBS:linear
-LIBS:regul
-LIBS:74xx
-LIBS:cmos4000
-LIBS:adc-dac
-LIBS:memory
-LIBS:xilinx
-LIBS:special
-LIBS:microcontrollers
-LIBS:dsp
-LIBS:microchip
-LIBS:analog_switches
-LIBS:motorola
-LIBS:texas
-LIBS:intel
-LIBS:audio
-LIBS:interface
-LIBS:digital-audio
-LIBS:philips
-LIBS:display
-LIBS:cypress
-LIBS:siliconi
-LIBS:opto
-LIBS:atmel
-LIBS:contrib
-LIBS:valves
-LIBS:armory
-LIBS:armory-cache
-EELAYER 24 0
+EESchema Schematic File Version 4
+EELAYER 30 0
 EELAYER END
 $Descr A3 16535 11693
@@
 $EndDescr
 $Comp
-L MX53 U2
+L armory:MX53 U2
 U 4 1 53834A45
 P 1560 6320
@@
 DRAM_A8
 $Comp
-L R R15
+L armory-rescue:R R15
 U 1 1 53870145
 P 15500 5350
@@
 $EndComp
 $Comp
-L GND #PWR087
+L armory-rescue:GND #PWR087
 U 1 1 53870351
 P 15500 6500
@@
 $EndComp
 $Comp
-L C C90
+L armory-rescue:C C90
 U 1 1 5387046A
 P 15050 5350
@@
 $EndComp
 $Comp
-L C C89
+L armory-rescue:C C89
 U 1 1 53870475
 P 14900 6150
@@
 DDR_VREF
 $Comp
-L TST P3
+L armory-rescue:TST P3
 U 1 1 53870B46
 P 14600 5400
@@
 $EndComp
 $Comp
-L GND #PWR088
+L armory-rescue:GND #PWR088
 U 1 1 5390977F
 P 10850 9100
@@
 DRAM_SDODT0
 $Comp
-L R R29
+L armory-rescue:R R29
 U 1 1 5390703C
 P 5300 8250
@@
 $EndComp
 $Comp
-L GND #PWR089
+L armory-rescue:GND #PWR089
 U 1 1 53907105
 P 5300 8700
@@
 $EndComp
 $Comp
-L GND #PWR090
+L armory-rescue:GND #PWR090
 U 1 1 53907114
 P 5300 8700
@@
 $EndComp
 $Comp
-L R R27
+L armory-rescue:R R27
 U 1 1 539071C7
 P 4000 5250
@@
 $EndComp
 $Comp
-L GND #PWR091
+L armory-rescue:GND #PWR091
 U 1 1 539071CD
 P 4000 5700
@@
 $EndComp
 $Comp
-L GND #PWR092
+L armory-rescue:GND #PWR092
 U 1 1 539071D3
 P 4000 5700
@@
 PMIC_DDR_1V5
 $Comp
-L C C94
+L armory-rescue:C C94
 U 1 1 53908537
 P 13500 1700
@@
 $EndComp
 $Comp
-L C C95
+L armory-rescue:C C95
 U 1 1 53908556
 P 13800 1700
@@
 $EndComp
 $Comp
-L C C97
+L armory-rescue:C C97
 U 1 1 53908561
 P 14100 1700
@@
 $EndComp
 $Comp
-L C C99
+L armory-rescue:C C99
 U 1 1 5390858E
 P 14400 1700
@@
 $EndComp
 $Comp
-L C C101
+L armory-rescue:C C101
 U 1 1 53908599
 P 14700 1700
@@
 $EndComp
 $Comp
-L C C103
+L armory-rescue:C C103
 U 1 1 539085A4
 P 15000 1700
@@
 $EndComp
 $Comp
-L C C105
+L armory-rescue:C C105
 U 1 1 539085AF
 P 15300 1700
@@
 Connection ~ 13500 1200
 $Comp
-L GND #PWR093
+L armory-rescue:GND #PWR093
 U 1 1 53908C55
 P 15300 2200
@@
 PMIC_DDR_1V5
 $Comp
-L C C98
+L armory-rescue:C C98
 U 1 1 53909367
 P 14100 3150
@@
 $EndComp
 $Comp
-L C C102
+L armory-rescue:C C102
 U 1 1 5390937D
 P 14700 3150
@@
 $EndComp
 $Comp
-L C C106
+L armory-rescue:C C106
 U 1 1 53909393
 P 15300 3150
@@
 Connection ~ 13800 2650
 $Comp
-L GND #PWR094
+L armory-rescue:GND #PWR094
 U 1 1 539093A7
 P 15300 3650
@@
 Place near the VDDQ balls.
 $Comp
-L C C96
+L armory-rescue:C C96
 U 1 1 539093C2
 P 13800 3150
@@
 $EndComp
 $Comp
-L C C100
+L armory-rescue:C C100
 U 1 1 539093CD
 P 14400 3150
@@
 $EndComp
 $Comp
-L C C104
+L armory-rescue:C C104
 U 1 1 539093D8
 P 15000 3150
@@
 	13800 3450 15300 3450
 $Comp
-L C C91
+L armory-rescue:C C91
 U 1 1 539094E1
 P 5800 8100
@@
 $EndComp
 $Comp
-L C C93
+L armory-rescue:C C93
 U 1 1 53909500
 P 6100 8100
@@
 	5800 7150 5800 7900
 $Comp
-L GND #PWR095
+L armory-rescue:GND #PWR095
 U 1 1 5390971C
 P 5800 8600
@@
 	2550 6750 3300 6750
 $Comp
-L R R24
+L armory-rescue:R R24
 U 1 1 53C6BDEB
 P 15500 6150
@@
 DRAM_A14
 $Comp
-L MT41J256M16HA U4
+L armory:MT41J256M16HA U4
 U 1 1 53909770
 P 9200 4900
@@
 DRAM_A14
 $Comp
-L R R30
+L armory-rescue:R R30
 U 1 1 53F354E7
 P 14600 7650
