File: mark-one/USB.sch (KiCad schematic (older format))
At the start: 19 parts, among them U2 MX53

Commit message: made changes
Parts:
- C113, C114, C115, C116, C117, C76, C92: symbol C -> armory-rescue:C
- L7, L8: symbol INDUCTOR -> armory-rescue:INDUCTOR
- R28, R37, R38, R40, R41, R42, R43, R44, R57: symbol R -> armory-rescue:R
- U2: symbol MX53 -> armory:MX53
Changed lines of the file:
@@
-EESchema Schematic File Version 2
-LIBS:power
-LIBS:device
-LIBS:transistors
-LIBS:conn
-LIBS:linear
-LIBS:regul
-LIBS:74xx
-LIBS:cmos4000
-LIBS:adc-dac
-LIBS:memory
-LIBS:xilinx
-LIBS:special
-LIBS:microcontrollers
-LIBS:dsp
-LIBS:microchip
-LIBS:analog_switches
-LIBS:motorola
-LIBS:texas
-LIBS:intel
-LIBS:audio
-LIBS:interface
-LIBS:digital-audio
-LIBS:philips
-LIBS:display
-LIBS:cypress
-LIBS:siliconi
-LIBS:opto
-LIBS:atmel
-LIBS:contrib
-LIBS:valves
-LIBS:armory
-LIBS:armory-cache
-EELAYER 24 0
+EESchema Schematic File Version 4
+EELAYER 30 0
 EELAYER END
 $Descr A3 16535 11693
@@
 Freescale\nreserved.\n(M53UG)
 $Comp
-L R R28
+L armory-rescue:R R28
 U 1 1 538F5CEA
 P 10250 5400
@@
 $EndComp
 $Comp
-L GND #PWR070
+L armory-rescue:GND #PWR070
 U 1 1 538F5CF2
 P 10250 5850
@@
 	9850 4750 9350 4750
 $Comp
-L C C76
+L armory-rescue:C C76
 U 1 1 538F5E31
 P 7250 5450
@@
 $EndComp
 $Comp
-L GND #PWR071
+L armory-rescue:GND #PWR071
 U 1 1 538F5E37
 P 7250 5750
@@
 PMIC_SW4_3V3
 $Comp
-L INDUCTOR L7
+L armory-rescue:INDUCTOR L7
 U 1 1 53C505BA
 P 4600 4750
@@
 $EndComp
 $Comp
-L C C115
+L armory-rescue:C C115
 U 1 1 53C505D2
 P 5600 5050
@@
 	7150 4750 4900 4750
 $Comp
-L C C113
+L armory-rescue:C C113
 U 1 1 53C50763
 P 5200 5050
@@
 $EndComp
 $Comp
-L GND #PWR072
+L armory-rescue:GND #PWR072
 U 1 1 53C5077D
 P 5600 5350
@@
 $EndComp
 $Comp
-L GND #PWR073
+L armory-rescue:GND #PWR073
 U 1 1 53C50788
 P 5200 5350
@@
 Connection ~ 5600 4750
 $Comp
-L R R38
+L armory-rescue:R R38
 U 1 1 53C525CB
 P 11750 5400
@@
 $EndComp
 $Comp
-L R R37
+L armory-rescue:R R37
 U 1 1 53C5265E
 P 11750 4700
@@
 	11750 4950 11750 5150
 $Comp
-L GND #PWR074
+L armory-rescue:GND #PWR074
 U 1 1 53C52697
 P 11750 5850
@@
 	11750 3150 11750 4450
 $Comp
-L R R44
+L armory-rescue:R R44
 U 1 1 53C65C52
 P 11250 3700
@@
 $EndComp
 $Comp
-L C C117
+L armory-rescue:C C117
 U 1 1 53C65CBE
 P 11250 4350
@@
 $EndComp
 $Comp
-L GND #PWR075
+L armory-rescue:GND #PWR075
 U 1 1 53C65CDA
 P 11250 4650
@@
 Connection ~ 11250 4050
 $Comp
-L R R40
+L armory-rescue:R R40
 U 1 1 53C65E19
 P 3950 4750
@@
 	3600 4750 3700 4750
 $Comp
-L R R42
+L armory-rescue:R R42
 U 1 1 53C660B6
 P 6800 5250
@@
 	6350 5250 6550 5250
 $Comp
-L R R57
+L armory-rescue:R R57
 U 1 1 53D239AA
 P 10250 6200
@@
 $EndComp
 $Comp
-L GND #PWR076
+L armory-rescue:GND #PWR076
 U 1 1 53D239B0
 P 10250 6650
@@
 According to Freescale USB_H1_RREFEXT must\nbe connected for JTAG to work.
 $Comp
-L MX53 U2
+L armory:MX53 U2
 U 10 1 538352C5
 P 8400 5450
@@
 $EndComp
 $Comp
-L PWR_FLAG #FLG077
+L power:PWR_FLAG #FLG077
 U 1 1 5406978D
 P 7000 4650
@@
 Connection ~ 7000 4750
 $Comp
-L PWR_FLAG #FLG078
+L power:PWR_FLAG #FLG078
 U 1 1 5406981E
 P 7400 4950
@@
 Connection ~ 7400 5250
 $Comp
-L PWR_FLAG #FLG079
+L power:PWR_FLAG #FLG079
 U 1 1 5406A219
 P 10550 4800
@@
 	6350 3850 6350 5850
 $Comp
-L INDUCTOR L8
+L armory-rescue:INDUCTOR L8
 U 1 1 542A73D2
 P 4600 5650
@@
 $EndComp
 $Comp
-L C C116
+L armory-rescue:C C116
 U 1 1 542A73DD
 P 5600 5950
@@
 	4900 5650 7450 5650
 $Comp
-L C C114
+L armory-rescue:C C114
 U 1 1 542A73E9
 P 5200 5950
@@
 $EndComp
 $Comp
-L GND #PWR080
+L armory-rescue:GND #PWR080
 U 1 1 542A73EF
 P 5600 6250
@@
 $EndComp
 $Comp
-L GND #PWR081
+L armory-rescue:GND #PWR081
 U 1 1 542A73F5
 P 5200 6250
@@
 Connection ~ 5600 5650
 $Comp
-L R R41
+L armory-rescue:R R41
 U 1 1 542A7406
 P 3950 5650
@@
 Connection ~ 3600 4750
 $Comp
-L R R43
+L armory-rescue:R R43
 U 1 1 542A7536
 P 6800 5850
@@
 	7050 5850 7450 5850
 $Comp
-L C C92
+L armory-rescue:C C92
 U 1 1 542A75E0
 P 7250 6150
@@
 $EndComp
 $Comp
-L GND #PWR082
+L armory-rescue:GND #PWR082
 U 1 1 542A7609
 P 7250 6450
@@
 	7250 6350 7250 6450
 $Comp
-L PWR_FLAG #FLG083
+L power:PWR_FLAG #FLG083
 U 1 1 542A776F
 P 7600 6100
@@
 $EndComp
 $Comp
-L PWR_FLAG #FLG084
+L power:PWR_FLAG #FLG084
 U 1 1 542A777A
 P 6100 5500
