File: mark-one/boot.sch (KiCad schematic (older format))
At the start: 5 parts, among them U2 MX53

Commit message: made changes
Parts:
- R25, R32, R33, R34: symbol R -> armory-rescue:R
- U2: symbol MX53 -> armory:MX53
Changed lines of the file:
@@
-EESchema Schematic File Version 2
-LIBS:power
-LIBS:device
-LIBS:transistors
-LIBS:conn
-LIBS:linear
-LIBS:regul
-LIBS:74xx
-LIBS:cmos4000
-LIBS:adc-dac
-LIBS:memory
-LIBS:xilinx
-LIBS:special
-LIBS:microcontrollers
-LIBS:dsp
-LIBS:microchip
-LIBS:analog_switches
-LIBS:motorola
-LIBS:texas
-LIBS:intel
-LIBS:audio
-LIBS:interface
-LIBS:digital-audio
-LIBS:philips
-LIBS:display
-LIBS:cypress
-LIBS:siliconi
-LIBS:opto
-LIBS:atmel
-LIBS:contrib
-LIBS:valves
-LIBS:armory
-LIBS:armory-cache
-EELAYER 24 0
+EESchema Schematic File Version 4
+EELAYER 30 0
 EELAYER END
 $Descr A3 16535 11693
@@
 $EndDescr
 $Comp
-L MX53 U?
+L armory:MX53 U?
 U 5 1 53C625CC
 P 6550 5250
@@
 BT_CFG2_5
 $Comp
-L GND #PWR085
+L armory-rescue:GND #PWR085
 U 1 1 53C6261D
 P 8800 4500
@@
 PMIC_SW4_3V3
 $Comp
-L R R25
+L armory-rescue:R R25
 U 1 1 53C6262C
 P 9650 3750
@@
 Connection ~ 8800 2750
 $Comp
-L R R32
+L armory-rescue:R R32
 U 1 1 53C6263C
 P 9950 3750
@@
 Connection ~ 9950 3200
 $Comp
-L GND #PWR086
+L armory-rescue:GND #PWR086
 U 1 1 53C62646
 P 8800 7750
@@
 I2C1_SDA
 $Comp
-L R R33
+L armory-rescue:R R33
 U 1 1 53C6A47B
 P 10700 4750
@@
 $EndComp
 $Comp
-L R R34
+L armory-rescue:R R34
 U 1 1 53C6A486
 P 11000 4750
