File: mark-one/imx53-misc.sch (KiCad schematic (older format))
At the start: 21 parts, among them P10 TST, P11 TST, P12 TST, P13 TST, P6 TST, P8 TST, P9 TST, U2 MX53, X1 32.768kHz, X2 24MHz

Commit message: made changes
Parts:
- C111, C112, C84, C85, C86, C87: symbol C -> armory-rescue:C
- P10, P11, P12, P13, P6, P8, P9: symbol TST -> armory-rescue:TST
- R21, R22, R26, R35, R39: symbol R -> armory-rescue:R
- U2: symbol MX53 -> armory:MX53
- X1: symbol CRYSTAL -> armory-rescue:CRYSTAL
- X2: symbol CRYSTAL-24M -> armory:CRYSTAL-24M
Changed lines of the file:
@@
-EESchema Schematic File Version 2
-LIBS:power
-LIBS:device
-LIBS:transistors
-LIBS:conn
-LIBS:linear
-LIBS:regul
-LIBS:74xx
-LIBS:cmos4000
-LIBS:adc-dac
-LIBS:memory
-LIBS:xilinx
-LIBS:special
-LIBS:microcontrollers
-LIBS:dsp
-LIBS:microchip
-LIBS:analog_switches
-LIBS:motorola
-LIBS:texas
-LIBS:intel
-LIBS:audio
-LIBS:interface
-LIBS:digital-audio
-LIBS:philips
-LIBS:display
-LIBS:cypress
-LIBS:siliconi
-LIBS:opto
-LIBS:atmel
-LIBS:contrib
-LIBS:valves
-LIBS:armory
-LIBS:armory-cache
-EELAYER 24 0
+EESchema Schematic File Version 4
+EELAYER 30 0
 EELAYER END
 $Descr A3 16535 11693
@@
 NoConn ~ 10050 6550
 $Comp
-L GND #PWR051
+L armory-rescue:GND #PWR051
 U 1 1 533C7F7B
 P 10650 8250
@@
 $EndComp
 $Comp
-L GND #PWR052
+L armory-rescue:GND #PWR052
 U 1 1 533C7F8A
 P 12350 8250
@@
 $EndComp
 $Comp
-L C C84
+L armory-rescue:C C84
 U 1 1 533C7FC2
 P 7400 6250
@@
 $EndComp
 $Comp
-L R R21
+L armory-rescue:R R21
 U 1 1 533AEA7B
 P 5550 5900
@@
 $EndComp
 $Comp
-L GND #PWR053
+L armory-rescue:GND #PWR053
 U 1 1 533AEACF
 P 5850 6450
@@
 $EndComp
 $Comp
-L GND #PWR054
+L armory-rescue:GND #PWR054
 U 1 1 533AEADE
 P 5550 6450
@@
 Boot Mode: [0, 0] Internal Boot\nIf errors occur -> Serial Downloader Mode\n\nfloating: BOOT_MODE0, BOOT_MODE1\n  IMX53IEC Rev. 6, 03/2013, pg 30\n  Recommendation 35: internal pull-down on BOOT_MODE0 and BOOT_MODE1\n\nfloating: TEST_MODE\n  IMX53IEC Rev. 6, 03/2013, pg 30\n  Recommendation 17
 $Comp
-L C C85
+L armory-rescue:C C85
 U 1 1 53846604
 P 7400 6850
@@
 $EndComp
 $Comp
-L R R22
+L armory-rescue:R R22
 U 1 1 53846713
 P 5850 6000
@@
 $EndComp
 $Comp
-L C C86
+L armory-rescue:C C86
 U 1 1 53846AA0
 P 10650 8050
@@
 $EndComp
 $Comp
-L C C87
+L armory-rescue:C C87
 U 1 1 53846B60
 P 12350 8050
@@
 $EndComp
 $Comp
-L GND #PWR055
+L armory-rescue:GND #PWR055
 U 1 1 5388331A
 P 7100 7100
@@
 $EndComp
 $Comp
-L GND #PWR056
+L armory-rescue:GND #PWR056
 U 1 1 5390A1BA
 P 10950 8050
@@
 $EndComp
 $Comp
-L R R26
+L armory-rescue:R R26
 U 1 1 53BD3F54
 P 7750 2900
@@
 CKIH2
 $Comp
-L C C112
+L armory-rescue:C C112
 U 1 1 53C4F939
 P 7750 3550
@@
 $EndComp
 $Comp
-L GND #PWR057
+L armory-rescue:GND #PWR057
 U 1 1 53C4F93F
 P 7750 3850
@@
 $EndComp
 $Comp
-L R R35
+L armory-rescue:R R35
 U 1 1 53C4F9E2
 P 7250 2900
@@
 $EndComp
 $Comp
-L C C111
+L armory-rescue:C C111
 U 1 1 53C4F9F9
 P 7250 3550
@@
 $EndComp
 $Comp
-L GND #PWR058
+L armory-rescue:GND #PWR058
 U 1 1 53C4FAE4
 P 7250 3850
@@
 NoConn ~ 8140 5350
 $Comp
-L R R39
+L armory-rescue:R R39
 U 1 1 53C64427
 P 11550 7000
@@
 $EndComp
 $Comp
-L GND #PWR059
+L armory-rescue:GND #PWR059
 U 1 1 53C6B2C6
 P 12250 7350
@@
 MX53_XTAL
 $Comp
-L MX53 U2
+L armory:MX53 U2
 U 3 1 533C7F2F
 P 9100 5050
@@
 Connection ~ 10650 7700
 $Comp
-L CRYSTAL X1
+L armory-rescue:CRYSTAL X1
 U 1 1 53C6B178
 P 7750 6550
@@
 $EndComp
 $Comp
-L CRYSTAL-24M X2
+L armory:CRYSTAL-24M X2
 U 1 1 53C7998D
 P 11550 7650
@@
 NoConn ~ 8140 4500
 $Comp
-L TST P8
+L armory-rescue:TST P8
 U 1 1 54185BE1
 P 10200 3850
@@
 $EndComp
 $Comp
-L TST P9
+L armory-rescue:TST P9
 U 1 1 54185BE7
 P 10400 3850
@@
 $EndComp
 $Comp
-L TST P10
+L armory-rescue:TST P10
 U 1 1 54185BF2
 P 10600 3850
@@
 $EndComp
 $Comp
-L TST P11
+L armory-rescue:TST P11
 U 1 1 54185BFD
 P 10800 3850
@@
 $EndComp
 $Comp
-L TST P12
+L armory-rescue:TST P12
 U 1 1 54185C08
 P 11000 3850
@@
 Connection ~ 11000 4350
 $Comp
-L TST P13
+L armory-rescue:TST P13
 U 1 1 54185D44
 P 11200 3850
@@
 Connection ~ 11200 4450
 $Comp
-L TST P6
+L armory-rescue:TST P6
 U 1 1 54185D92
 P 10000 3400
