File: mark-one/imx53-power.sch (KiCad schematic (older format))
At the start: 63 parts, among them P1 TST, P2 TST, P5 TST, U2 MX53

Commit message: made changes
Parts:
- C20, C21, C22, C23, C24, C25, C26, C27, C28, C29, C30, C31, C32, C33, C34, C35, C36, C37, C38, C39, C40, C41, C42, C43, C44, C45, C46, C47, C48, C49, C50, C51, C52, C53, C54, C55, C56, C57, C58, C59, C60, C61, C62, C63, C64, C65, C66, C67, C68, C69, C70, C71, C72, C73, C74, C75, C81, C82: symbol C -> armory-rescue:C
- L5: symbol INDUCTOR -> armory-rescue:INDUCTOR
- P1, P2, P5: symbol TST -> armory-rescue:TST
- U2: symbol MX53 -> armory:MX53
