File: mark-one/interfaces.sch (KiCad schematic (older format))
At the start: 9 parts, among them J1 MICRO_SD_HINGE, P4 CONN_01X07, U2 MX53

Commit message: made changes
Parts:
- C107, C108: symbol C -> armory-rescue:C
- D1: symbol LED -> armory-rescue:LED
- J1: symbol MICRO_SD_HINGE -> armory:MICRO_SD_HINGE
- P4: symbol CONN_01X07 -> armory:CONN_01X07
- R16, R31, R45: symbol R -> armory-rescue:R
- U2: symbol MX53 -> armory:MX53
Changed lines of the file:
@@
-EESchema Schematic File Version 2
-LIBS:power
-LIBS:device
-LIBS:transistors
-LIBS:conn
-LIBS:linear
-LIBS:regul
-LIBS:74xx
-LIBS:cmos4000
-LIBS:adc-dac
-LIBS:memory
-LIBS:xilinx
-LIBS:special
-LIBS:microcontrollers
-LIBS:dsp
-LIBS:microchip
-LIBS:analog_switches
-LIBS:motorola
-LIBS:texas
-LIBS:intel
-LIBS:audio
-LIBS:interface
-LIBS:digital-audio
-LIBS:philips
-LIBS:display
-LIBS:cypress
-LIBS:siliconi
-LIBS:opto
-LIBS:atmel
-LIBS:contrib
-LIBS:valves
-LIBS:armory
-LIBS:armory-cache
-EELAYER 24 0
+EESchema Schematic File Version 4
+EELAYER 30 0
 EELAYER END
 $Descr A3 16535 11693
@@
 $EndDescr
 $Comp
-L MX53 U2
+L armory:MX53 U2
 U 7 1 53722D0E
 P 2410 3750
@@
 PMIC_SW4_3V3
 $Comp
-L MICRO_SD_HINGE J1
+L armory:MICRO_SD_HINGE J1
 U 1 1 53723105
 P 8770 2460
@@
 $EndComp
 $Comp
-L GND #PWR060
+L armory-rescue:GND #PWR060
 U 1 1 53B52B70
 P 6795 1960
@@
 $EndComp
 $Comp
-L C C107
+L armory-rescue:C C107
 U 1 1 53B52C94
 P 6795 1710
@@
 $EndComp
 $Comp
-L C C108
+L armory-rescue:C C108
 U 1 1 53B52D21
 P 7145 1710
@@
 $EndComp
 $Comp
-L GND #PWR061
+L armory-rescue:GND #PWR061
 U 1 1 53B52D59
 P 7145 1960
@@
 Place the capacitors near\nthe SD connector.
 $Comp
-L GND #PWR062
+L armory-rescue:GND #PWR062
 U 1 1 53B52E55
 P 8720 3610
@@
 $EndComp
 $Comp
-L R R31
+L armory-rescue:R R31
 U 1 1 53B532AD
 P 6420 1735
@@
 $EndComp
 $Comp
-L R R45
+L armory-rescue:R R45
 U 1 1 53C68F69
 P 6420 2460
@@
 SD1_CMD
 $Comp
-L MX53 U?
+L armory:MX53 U?
 U 6 1 5460C738
 P 10790 6950
@@
 NoConn ~ 9840 8550
 $Comp
-L GND #PWR063
+L armory-rescue:GND #PWR063
 U 1 1 5460C766
 P 7340 7150
@@
 GPIO5_30
 $Comp
-L CONN_01X07 P4
+L armory:CONN_01X07 P4
 U 1 1 5460C78E
 P 6940 7650
@@
 $EndComp
 $Comp
-L LED D1
+L armory-rescue:LED D1
 U 1 1 5460C799
 P 12840 4850
@@
 $EndComp
 $Comp
-L R R16
+L armory-rescue:R R16
 U 1 1 5460C7A5
 P 12840 5500
