File: mark-one/pmic.sch (KiCad schematic (older format))
At the start: 44 parts, among them U1 LTC3589, U3 NCP1529

Commit message: made changes
Parts:
- added C? (x2): 22uF, SM0603, symbol armory-rescue:C
- added C? (x3): 10pF, SM0402, symbol armory-rescue:C
- added L?: 2.2uH, VLS252012ET, symbol armory-rescue:INDUCTOR
- added R? (x2): 158k, SM0201, symbol armory-rescue:R
- added R? (x2): 100k, SM0201, symbol armory-rescue:R
- added R?: 180k, SM0201, symbol armory-rescue:R
- added R?: 511k, SM0201, symbol armory-rescue:R
- added R?: 191k, SM0201, symbol armory-rescue:R
- added R?: 270k, SM0201, symbol armory-rescue:R
- C1, C10, C109, C11, C110, C12, C13, C14, C15, C16, C17, C18, C19, C2, C3, C4, C5, C6, C7, C77, C78, C8, C9: symbol C -> armory-rescue:C
- L1, L2, L3, L4, L6: symbol INDUCTOR -> armory-rescue:INDUCTOR
- R1, R10, R11, R12, R13, R2, R23, R3, R4, R5, R6, R7, R8, R9: symbol R -> armory-rescue:R
- U1: symbol LTC3589 -> armory:LTC3589
- U3: symbol NCP1529 -> armory-rescue:NCP1529
Connections:
- wire segments 110 -> 205
Other:
- moved on the sheet: C2, C7, C8, C9, R3, R4
