File: mark-one/unused.sch (KiCad schematic (older format))
At the start: 3 parts, among them U2 MX53

Commit message: made changes
Parts:
- C88: symbol C -> armory-rescue:C
- R14: symbol R -> armory-rescue:R
- U2: symbol MX53 -> armory:MX53
Changed lines of the file:
@@
-EESchema Schematic File Version 2
-LIBS:power
-LIBS:device
-LIBS:transistors
-LIBS:conn
-LIBS:linear
-LIBS:regul
-LIBS:74xx
-LIBS:cmos4000
-LIBS:adc-dac
-LIBS:memory
-LIBS:xilinx
-LIBS:special
-LIBS:microcontrollers
-LIBS:dsp
-LIBS:microchip
-LIBS:analog_switches
-LIBS:motorola
-LIBS:texas
-LIBS:intel
-LIBS:audio
-LIBS:interface
-LIBS:digital-audio
-LIBS:philips
-LIBS:display
-LIBS:cypress
-LIBS:siliconi
-LIBS:opto
-LIBS:atmel
-LIBS:contrib
-LIBS:valves
-LIBS:armory
-LIBS:armory-cache
-EELAYER 24 0
+EESchema Schematic File Version 4
+EELAYER 30 0
 EELAYER END
 $Descr A3 16535 11693
@@
 $EndDescr
 $Comp
-L MX53 U2
+L armory:MX53 U2
 U 8 1 53834052
 P 9170 3930
@@
 NoConn ~ 8220 4230
 $Comp
-L GND #PWR064
+L armory-rescue:GND #PWR064
 U 1 1 538340B8
 P 7870 3830
@@
 $EndComp
 $Comp
-L GND #PWR065
+L armory-rescue:GND #PWR065
 U 1 1 538340C5
 P 7720 3730
@@
 	7870 3730 7870 3830
 $Comp
-L GND #PWR066
+L armory-rescue:GND #PWR066
 U 1 1 538340D0
 P 7720 4030
@@
 $EndComp
 $Comp
-L GND #PWR067
+L armory-rescue:GND #PWR067
 U 1 1 538340D6
 P 7870 4130
@@
 	7870 4030 7870 4130
 $Comp
-L MX53 U2
+L armory:MX53 U2
 U 9 1 538340EA
 P 12730 4020
@@
 NoConn ~ 11780 4120
 $Comp
-L MX53 U2
+L armory:MX53 U2
 U 1 1 53834141
 P 5110 4800
@@
 PMIC_SW3_2V5
 $Comp
-L C C88
+L armory-rescue:C C88
 U 1 1 538341C5
 P 4060 4150
@@
 Connection ~ 4060 3800
 $Comp
-L GND #PWR068
+L armory-rescue:GND #PWR068
 U 1 1 53834223
 P 4060 4500
@@
 Connection ~ 3460 3700
 $Comp
-L R R14
+L armory-rescue:R R14
 U 1 1 53C3B046
 P 3710 3800
@@
 NoConn ~ 13680 4320
 $Comp
-L PWR_FLAG #FLG069
+L power:PWR_FLAG #FLG069
 U 1 1 540688C4
 P 3710 4200
