File: mark-one/armory.kicad_pcb (KiCad board)
At the start: 8 copper layers, 65.6 x 19.6 mm, 184 parts, among them J1 MICRO_SD_HINGE, J2 USB_A_PLUG, P1 TST, P10 TST, P11 TST, P12 TST, P13 TST, P2 TST, P3 TST, P4 CONN_01X07, P5 TST, P6 TST, P8 TST, P9 TST, U2 MX53, U3 NCP1529, U4 MT41K256M16HA, U5 TPD2E001DRLR, X1 32.768kHz, X2 24MHz

Commit message: made changes
Parts:
- removed C11: 22uF, smd:SM0603
- removed L4: 2.2uH, smd:VLS252012ET
- removed R13: 47k, smd:SM0201
- added P4: CONN_01X07, connectors:pinhead-1X7, F.Cu at (177.2, 95.4)
- added P4: CONN_01X07, connectors:pinhead-1X7, F.Cu at (174.7, 95.4)
- added P4: CONN_01X07, connectors:pinhead-1X7, F.Cu at (172.2, 95.4)
Routing:
- net /Interfaces/GPIO5_30: track 39.8 -> 10.8 mm
- net /Interfaces/UART1_RX: track 43.2 -> 26.9 mm
- net /Interfaces/UART1_TX: track 42.2 -> 26.3 mm
- net /Interfaces/GPIO5_27: track 45.1 -> 37.3 mm
- removed copper zone on F.Cu, net GND
- removed copper zone on SIGNAL_1, net GND

Commit message: modified zones
Changed lines of the file:
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@@
   (layers
     (0 TOP signal)
-    (1 GND_1 power hide)
+    (1 GND_1 power)
     (2 SIGNAL_1 signal)
-    (3 GND_POWER_1 power hide)
-    (4 GND_POWER_2 power hide)
-    (5 SIGNAL_2 signal hide)
-    (6 GND_2 power hide)
-    (31 BOTTOM signal hide)
+    (3 GND_POWER_1 power)
+    (4 GND_POWER_2 power)
+    (5 SIGNAL_2 signal)
+    (6 GND_2 power)
+    (31 BOTTOM signal)
     (32 B.Adhes user)
     (33 F.Adhes user)
@@
     (polygon
       (pts
-        (xy 170.2 105.1) (xy 113.2 105.1) (xy 113.2 85.7) (xy 170.2 85.7)
+        (xy 172.57 105.1) (xy 115.57 105.1) (xy 115.57 85.7) (xy 172.57 85.7)
       )
     )
@@
     (polygon
       (pts
-        (xy 170.2 105.1) (xy 104 105.1) (xy 104 85.7) (xy 170.2 85.7)
+        (xy 167.8 104.765198) (xy 101.6 104.765198) (xy 101.6 85.365198) (xy 167.8 85.365198)
       )
     )
@@
     (polygon
       (pts
-        (xy 169.4 91.4) (xy 166.15 91.4) (xy 166.15 87.75) (xy 144.8 87.75) (xy 144.8 86.4)
-        (xy 138.425 86.4) (xy 138.425 87.4) (xy 136.8 87.4) (xy 136.8 86.4) (xy 125.3 86.4)
-        (xy 125.3 88.225) (xy 127.2 88.225) (xy 127.2 90.55) (xy 126.25 90.55) (xy 126.25 92)
-        (xy 127.2 92) (xy 127.2 94.1) (xy 124.2 94.1) (xy 124.2 96.6) (xy 123.175 96.6)
-        (xy 123.175 95.575) (xy 119.1 95.575) (xy 119.1 95.075) (xy 119.1 91.4) (xy 123 91.4)
-        (xy 123 85.8) (xy 169.4 85.8)
+        (xy 169.358802 98.9) (xy 166.108802 98.9) (xy 166.108802 95.25) (xy 144.758802 95.25) (xy 144.758802 93.9)
+        (xy 138.383802 93.9) (xy 138.383802 94.9) (xy 136.758802 94.9) (xy 136.758802 93.9) (xy 125.258802 93.9)
+        (xy 125.258802 95.725) (xy 127.158802 95.725) (xy 127.158802 98.05) (xy 126.208802 98.05) (xy 126.208802 99.5)
+        (xy 127.158802 99.5) (xy 127.158802 101.6) (xy 124.158802 101.6) (xy 124.158802 104.1) (xy 123.133802 104.1)
+        (xy 123.133802 103.075) (xy 119.058802 103.075) (xy 119.058802 102.575) (xy 119.058802 98.9) (xy 122.958802 98.9)
+        (xy 122.958802 93.3) (xy 169.358802 93.3)
       )
     )
@@
     (polygon
       (pts
-        (xy 164.625 92.775) (xy 161.175 92.775) (xy 161.175 94.8) (xy 162.775 94.8) (xy 162.775 103.375)
-        (xy 147.2 103.375) (xy 147.2 85.75) (xy 164.625 85.75)
+        (xy 167.64 92.775) (xy 164.19 92.775) (xy 164.19 94.8) (xy 165.79 94.8) (xy 165.79 103.375)
+        (xy 150.215 103.375) (xy 150.215 85.75) (xy 167.64 85.75)
       )
     )

Commit message: changes
Parts:
- removed C105: 10uF, smd:SM0603
- added REF**: CP_Elec_3x5.4, Capacitor_SMD:CP_Elec_3x5.4, F.Cu at (101.6, 102.9)
- moved L6 6.03 mm to (119.4, 104.1)
Routing:
- removed copper zone on GND_POWER_2, net PMIC_SW4_3V3
Changed lines of the file:
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@@
   (layers
     (0 TOP signal)
-    (1 GND_1 power)
+    (1 GND_1 power hide)
     (2 SIGNAL_1 signal)
     (3 GND_POWER_1 power)
@@
     (add_net PMIC_SW4_3V3)
   )
+  (module Capacitor_SMD:CP_Elec_3x5.4 (layer TOP)
+    (at 101.6 102.87)
+    (descr "SMD capacitor, aluminum electrolytic, Nichicon, 3.0x5.4mm")
+    (tags "capacitor electrolytic")
+    (attr smd)
+    (fp_text reference REF** (at 0 -2.7) (layer F.SilkS)
+      (effects (font (size 1 1) (thickness 0.15)))
+    )
+    (fp_text value CP_Elec_3x5.4 (at 0 2.7) (layer F.Fab)
+      (effects (font (size 1 1) (thickness 0.15)))
+    )
+    (fp_text user %R (at 0 0) (layer F.Fab)
+      (effects (font (size 0.6 0.6) (thickness 0.09)))
+    )
+    (fp_line (start -2.85 1.05) (end -1.78 1.05) (layer F.CrtYd) (width 0.05))
+    (fp_line (start -2.85 -1.05) (end -2.85 1.05) (layer F.CrtYd) (width 0.05))
+    (fp_line (start -1.78 -1.05) (end -2.85 -1.05) (layer F.CrtYd) (width 0.05))
+    (fp_line (start -1.78 -1.05) (end -0.93 -1.9) (layer F.CrtYd) (width 0.05))
+    (fp_line (start -1.78 1.05) (end -0.93 1.9) (layer F.CrtYd) (width 0.05))
+    (fp_line (start -0.93 -1.9) (end 1.9 -1.9) (layer F.CrtYd) (width 0.05))
+    (fp_line (start -0.93 1.9) (end 1.9 1.9) (layer F.CrtYd) (width 0.05))
+    (fp_line (start 1.9 1.05) (end 1.9 1.9) (layer F.CrtYd) (width 0.05))
+    (fp_line (start 2.85 1.05) (end 1.9 1.05) (layer F.CrtYd) (width 0.05))
+    (fp_line (start 2.85 -1.05) (end 2.85 1.05) (layer F.CrtYd) (width 0.05))
+    (fp_line (start 1.9 -1.05) (end 2.85 -1.05) (layer F.CrtYd) (width 0.05))
+    (fp_line (start 1.9 -1.9) (end 1.9 -1.05) (layer F.CrtYd) (width 0.05))
+    (fp_line (start -2.1875 -1.6225) (end -2.1875 -1.2475) (layer F.SilkS) (width 0.12))
+    (fp_line (start -2.375 -1.435) (end -2 -1.435) (layer F.SilkS) (width 0.12))
+    (fp_line (start -1.570563 1.06) (end -0.870563 1.76) (layer F.SilkS) (width 0.12))
+    (fp_line (start -1.570563 -1.06) (end -0.870563 -1.76) (layer F.SilkS) (width 0.12))
+    (fp_line (start -0.870563 1.76) (end 1.76 1.76) (layer F.SilkS) (width 0.12))
+    (fp_line (start -0.870563 -1.76) (end 1.76 -1.76) (layer F.SilkS) (width 0.12))
+    (fp_line (start 1.76 -1.76) (end 1.76 -1.06) (layer F.SilkS) (width 0.12))
+    (fp_line (start 1.76 1.76) (end 1.76 1.06) (layer F.SilkS) (width 0.12))
+    (fp_line (start -0.960469 -0.95) (end -0.960469 -0.65) (layer F.Fab) (width 0.1))
+    (fp_line (start -1.110469 -0.8) (end -0.810469 -0.8) (layer F.Fab) (width 0.1))
+    (fp_line (start -1.65 0.825) (end -0.825 1.65) (layer F.Fab) (width 0.1))
+    (fp_line (start -1.65 -0.825) (end -0.825 -1.65) (layer F.Fab) (width 0.1))
+    (fp_line (start -1.65 -0.825) (end -1.65 0.825) (layer F.Fab) (width 0.1))
+    (fp_line (start -0.825 1.65) (end 1.65 1.65) (layer F.Fab) (width 0.1))
+    (fp_line (start -0.825 -1.65) (end 1.65 -1.65) (layer F.Fab) (width 0.1))
+    (fp_line (start 1.65 -1.65) (end 1.65 1.65) (layer F.Fab) (width 0.1))
+    (fp_circle (center 0 0) (end 1.5 0) (layer F.Fab) (width 0.1))
+    (pad 2 smd roundrect (at 1.5 0) (size 2.2 1.6) (layers TOP F.Paste F.Mask) (roundrect_rratio 0.15625))
+    (pad 1 smd roundrect (at -1.5 0) (size 2.2 1.6) (layers TOP F.Paste F.Mask) (roundrect_rratio 0.15625))
+    (model ${KISYS3DMOD}/Capacitor_SMD.3dshapes/CP_Elec_3x5.4.wrl
+      (at (xyz 0 0 0))
+      (scale (xyz 1 1 1))
+      (rotate (xyz 0 0 0))
+    )
+  )
   (module connectors:usb-PCB (layer TOP)
     (at 104.1 95.4 270)
@@
   )
   (module smd:SM0603 (layer TOP)
-    (at 165.2 99.21 90)
-    (attr smd)
-    (fp_text reference C105 (at 0 0.03556 90) (layer F.SilkS)
-      (effects (font (size 0.508 0.4572) (thickness 0.1143)))
-    )
-    (fp_text value 10uF (at 0.08636 0.04064 90) (layer F.SilkS) hide
-      (effects (font (size 0.508 0.4572) (thickness 0.1143)))
-    )
-    (fp_line (start -1.143 -0.635) (end 1.143 -0.635) (layer F.SilkS) (width 0.127))
-    (fp_line (start 1.143 -0.635) (end 1.143 0.635) (layer F.SilkS) (width 0.127))
-    (fp_line (start 1.143 0.635) (end -1.143 0.635) (layer F.SilkS) (width 0.127))
-    (fp_line (start -1.143 0.635) (end -1.143 -0.635) (layer F.SilkS) (width 0.127))
-    (pad 1 smd rect (at -0.762 0 90) (size 0.635 1.143) (layers TOP F.Paste F.Mask)
-      (net 59 PMIC_DDR_1V5))
-    (pad 2 smd rect (at 0.762 0 90) (size 0.635 1.143) (layers TOP F.Paste F.Mask)
-      (net 1 GND))
-    (model smd\resistors\R0603.wrl
-      (offset (xyz 0 0 0.02539999961853028))
-      (scale (xyz 0.5 0.5 0.5))
-      (rotate (xyz 0 0 0))
-    )
-  )
-  (module smd:SM0603 (layer TOP)
     (at 164.175 89.525)
     (attr smd)
@@
   )
   (module smd:VLS252012ET (layer TOP)
-    (at 125.24 102.73)
+    (at 119.38 104.14)
     (attr smd)
     (fp_text reference L6 (at 0.05588 -0.01016) (layer F.SilkS)
@@
     (polygon
       (pts
-        (xy 172.57 105.1) (xy 115.57 105.1) (xy 115.57 85.7) (xy 172.57 85.7)
+        (xy 153.52 105.1) (xy 96.52 105.1) (xy 96.52 85.7) (xy 153.52 85.7)
       )
     )
@@
     (polygon
       (pts
-        (xy 167.8 104.765198) (xy 101.6 104.765198) (xy 101.6 85.365198) (xy 167.8 85.365198)
-      )
-    )
-  )
-  (zone (net 55) (net_name PMIC_SW4_3V3) (layer GND_POWER_2) (hatch edge 0.508)
-    (connect_pads (clearance 0.127))
-    (min_thickness 0.127)
-    (fill (arc_segments 16) (thermal_gap 0.254) (thermal_bridge_width 0.4064))
-    (polygon
-      (pts
-        (xy 139.7 99.2) (xy 138.7 99.2) (xy 138.7 100.1) (xy 133.1 100.1) (xy 133.1 101)
-        (xy 131.4 101) (xy 117.45 101) (xy 117.45 88.6) (xy 121.3 88.6) (xy 121.3 90.75)
-        (xy 118.4 90.75) (xy 118.4 96.05) (xy 122.6 96.05) (xy 122.6 99) (xy 125 99)
-        (xy 130.725 99) (xy 130.725 97.6) (xy 135.2 97.6) (xy 135.2 96.3) (xy 135.8 96.3)
-        (xy 135.8 98.7) (xy 139.7 98.7)
+        (xy 170.2 105.1) (xy 104 105.1) (xy 104 85.7) (xy 170.2 85.7)
       )
     )
@@
     (polygon
       (pts
-        (xy 169.358802 98.9) (xy 166.108802 98.9) (xy 166.108802 95.25) (xy 144.758802 95.25) (xy 144.758802 93.9)
-        (xy 138.383802 93.9) (xy 138.383802 94.9) (xy 136.758802 94.9) (xy 136.758802 93.9) (xy 125.258802 93.9)
-        (xy 125.258802 95.725) (xy 127.158802 95.725) (xy 127.158802 98.05) (xy 126.208802 98.05) (xy 126.208802 99.5)
-        (xy 127.158802 99.5) (xy 127.158802 101.6) (xy 124.158802 101.6) (xy 124.158802 104.1) (xy 123.133802 104.1)
-        (xy 123.133802 103.075) (xy 119.058802 103.075) (xy 119.058802 102.575) (xy 119.058802 98.9) (xy 122.958802 98.9)
-        (xy 122.958802 93.3) (xy 169.358802 93.3)
+        (xy 169.4 91.4) (xy 166.15 91.4) (xy 166.15 87.75) (xy 144.8 87.75) (xy 144.8 86.4)
+        (xy 138.425 86.4) (xy 138.425 87.4) (xy 136.8 87.4) (xy 136.8 86.4) (xy 125.3 86.4)
+        (xy 125.3 88.225) (xy 127.2 88.225) (xy 127.2 90.55) (xy 126.25 90.55) (xy 126.25 92)
+        (xy 127.2 92) (xy 127.2 94.1) (xy 124.2 94.1) (xy 124.2 96.6) (xy 123.175 96.6)
+        (xy 123.175 95.575) (xy 119.1 95.575) (xy 119.1 95.075) (xy 119.1 91.4) (xy 123 91.4)
+        (xy 123 85.8) (xy 169.4 85.8)
       )
     )
@@
     (polygon
       (pts
-        (xy 167.64 92.775) (xy 164.19 92.775) (xy 164.19 94.8) (xy 165.79 94.8) (xy 165.79 103.375)
-        (xy 150.215 103.375) (xy 150.215 85.75) (xy 167.64 85.75)
+        (xy 164.625 92.775) (xy 161.175 92.775) (xy 161.175 94.8) (xy 162.775 94.8) (xy 162.775 103.375)
+        (xy 147.2 103.375) (xy 147.2 85.75) (xy 164.625 85.75)
       )
     )
